Commit message: Modified path planning by adding both heading and strafe variations, fixed issues with optitrack usage

File: src/rb2301_gz/urdf/nanocar_description.urdf (robot description, URDF)
Before this commit: robot NanoCar, 9 links, 8 joints
Links:
- link back_left_wheel_link: geometry collision mesh filename=package://rb2301_gz/meshes/nanocar/back_left_wheel_link.STL; visual mesh filename=package://rb2301_gz/meshes/nanocar/back_left_wheel_link.STL
- link back_right_wheel_link: geometry collision mesh filename=package://rb2301_gz/meshes/nanocar/back_right_wheel_link.STL; visual mesh filename=package://rb2301_gz/meshes/nanocar/back_right_wheel_link.STL
- link base_camera_link: geometry collision mesh filename=package://rb2301_gz/meshes/nanocar/base_camera_link.STL; visual mesh filename=package://rb2301_gz/meshes/nanocar/base_camera_link.STL
- link base_laser_link: geometry collision mesh filename=package://rb2301_gz/meshes/nanocar/base_laser_link.STL; visual mesh filename=package://rb2301_gz/meshes/nanocar/base_laser_link.STL
- link base_link: geometry collision mesh filename=package://rb2301_gz/meshes/nanocar/base_link.STL; visual mesh filename=package://rb2301_gz/meshes/nanocar/base_link.STL
- link front_left_wheel_link: geometry collision mesh filename=package://rb2301_gz/meshes/nanocar/front_left_wheel_link.STL; visual mesh filename=package://rb2301_gz/meshes/nanocar/front_left_wheel_link.STL
- link front_right_wheel_link: geometry collision mesh filename=package://rb2301_gz/meshes/nanocar/front_right_wheel_link.S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; visual mesh filename=package://rb2301_gz/meshes/nanocar/front_right_wheel_link.S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
- link imu_link: geometry collision mesh filename=package://rb2301_gz/meshes/nanocar/imu.STL; visual mesh filename=package://rb2301_gz/meshes/nanocar/imu.STL
